File: knobber/MCU.kicad_sch (KiCad schematic)
At the start: 16 parts, among them J801 Conn_01x04_Socket, J802 Micro_SD_Card, U801 BMD-340-A-R, U802 ESD224DQA

Commit message: Updated schematic & PCB
Parts:
- J801: value Conn_01x04_Socket -> SWD
Other:
- moved on the sheet: C801, C802, C803, C804, C805, J801, J802, R801, R802, R803, R804, R805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
