File: knobber/Motor_driver.kicad_sch (KiCad schematic)
At the start: 17 parts, among them U601 TMC6300-LA-T, U602 LMV321

Commit message: Updated schematic & PCB
Parts:
- added TP601: MOT_UH, TestPoint:TestPoint_Pad_D1.0mm, symbol Connector:TestPoint
- added TP602: MOT_UL, TestPoint:TestPoint_Pad_D1.0mm, symbol Connector:TestPoint
- added TP603: MOT_VH, TestPoint:TestPoint_Pad_D1.0mm, symbol Connector:TestPoint
- added TP604: MOT_VL, TestPoint:TestPoint_Pad_D1.0mm, symbol Connector:TestPoint
- added TP605: MOT_WH, TestPoint:TestPoint_Pad_D1.0mm, symbol Connector:TestPoint
- added TP606: MOT_WL, TestPoint:TestPoint_Pad_D1.0mm, symbol Connector:TestPoint
- added TP607: Cur_sens, TestPoint:TestPoint_Pad_D1.0mm, symbol Connector:TestPoint
- added TP608: MOT_DIAG, TestPoint:TestPoint_Pad_D1.0mm, symbol Connector:TestPoint
- added TP609: MOT_U, TestPoint:TestPoint_Pad_D1.0mm, symbol Connector:TestPoint
- added TP610: MOT_V, TestPoint:TestPoint_Pad_D1.0mm, symbol Connector:TestPoint
- added TP611: MOT_W, TestPoint:TestPoint_Pad_D1.0mm, symbol Connector:TestPoint
Connections:
- net MOT_DIAG: now also TP608.1
- net MOT_U: now also TP609.1
- net MOT_UH: now also TP601.1
- net MOT_UL: now also TP602.1
- net MOT_V: now also TP610.1
- net MOT_VH: now also TP603.1
- net MOT_VL: now also TP604.1
- net MOT_W: now also TP611.1
- net MOT_WH: now also TP605.1
- net MOT_WL: now also TP606.1
- net at R607.2, U601.16 (BRUV), U601.20 (BRW)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: now also TP607.1
Other:
- moved on the sheet: C601, C602, C603, C604, C605, C606, R601, R602, R603, R604, R605, R606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
