File: knobber/Switches.kicad_sch (KiCad schematic)
At the start: 82 parts, among them U701 SN74LV1T34DBV

Commit message: Updated schematic & PCB
Parts:
- added TP701: LED_DATA, TestPoint:TestPoint_Pad_D1.0mm, symbol Connector:TestPoint
Connections:
- net at LED701.3 (DIN), U701.4 (Y): now also TP701.1
Other:
- moved on the sheet: C701, C702, C703, C704, C705, C706, C707, C708, C709, C710, C711, C712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
