File: knobber/USB.kicad_sch (KiCad schematic)
At the start: 5 parts, among them J301 USB_C_Receptacle_USB2.0_16P

Commit message: Updated schematic & PCB
Other:
- moved on the sheet: C301, D301, J301, R301, R302
