File: knobber/knobber.kicad_pcb (KiCad board)
At the start: 4 copper layers, 170 x 110 mm, 165 parts, among them J101 BLDC, J301 USB_C_Receptacle_USB2.0_16P, J801 Conn_01x04_Socket, J802 Micro_SD_Card, J901 Conn_01x08_Socket, U201 SN74LV1T34DBV, U401 MT6701CT, U402 VEML7700-TT, U501 AP2112K-3.3, U601 TMC6300-LA-T, U602 LMV321, U701 SN74LV1T34DBV, U801 BMD-340-A-R, U802 ESD224DQA

Commit message: Updated schematic & PCB
Parts:
- added JP401: SolderJumper_3_Bridged12, Jumper:SolderJumper-3_P1.3mm_Bridged12_Pad1.0x1.5mm, F.Cu at (137.0, 99.5)
- added R403: 2.2k, Resistor_SMD:R_0603_1608Metric, F.Cu at (145.0, 104.4)
- added R404: 2.2k, Resistor_SMD:R_0603_1608Metric, F.Cu at (145.0, 106.2)
- added R405: 100k, Resistor_SMD:R_0603_1608Metric, F.Cu at (145.0, 107.9)
- added R406: 0, Resistor_SMD:R_0603_1608Metric, F.Cu at (145.0, 102.7)
- added TP201: LED_DATA, TestPoint:TestPoint_Pad_D1.0mm, F.Cu at (352.2, 183.2)
- added TP401: SDA, TestPoint:TestPoint_Pad_D1.0mm, F.Cu at (95.6, 56.8)
- added TP402: SCL, TestPoint:TestPoint_Pad_D1.0mm, F.Cu at (90.3, 56.8)
- added TP406: ENC__~{CS}, TestPoint:TestPoint_Pad_D1.0mm, F.Cu at (142.0, 102.7)
- added TP501: 5V, TestPoint:TestPoint_Pad_D1.0mm, F.Cu at (146.5, 57.2)
- added TP502: 3.3V, TestPoint:TestPoint_Pad_D1.0mm, F.Cu at (153.5, 57.2)
- added TP503: GND, TestPoint:TestPoint_Pad_D1.0mm, F.Cu at (153.5, 62.8)
- added TP601: MOT_UH, TestPoint:TestPoint_Pad_D1.0mm, F.Cu at (338.1, 169.1)
- added TP602: MOT_UL, TestPoint:TestPoint_Pad_D1.0mm, F.Cu at (338.1, 173.1)
- added TP603: MOT_VH, TestPoint:TestPoint_Pad_D1.0mm, F.Cu at (338.1, 177.2)
- added TP604: MOT_VL, TestPoint:TestPoint_Pad_D1.0mm, F.Cu at (338.1, 181.2)
- added TP605: MOT_WH, TestPoint:TestPoint_Pad_D1.0mm, F.Cu at (342.1, 169.1)
- added TP606: MOT_WL, TestPoint:TestPoint_Pad_D1.0mm, F.Cu at (342.1, 173.1)
- added TP607: Cur_sens, TestPoint:TestPoint_Pad_D1.0mm, F.Cu at (342.1, 177.2)
- added TP608: MOT_DIAG, TestPoint:TestPoint_Pad_D1.0mm, F.Cu at (342.1, 181.2)
- added TP609: MOT_U, TestPoint:TestPoint_Pad_D1.0mm, F.Cu at (346.2, 169.1)
- added TP610: MOT_V, TestPoint:TestPoint_Pad_D1.0mm, F.Cu at (346.2, 173.1)
- added TP611: MOT_W, TestPoint:TestPoint_Pad_D1.0mm, F.Cu at (346.2, 177.2)
- added TP701: LED_DATA, TestPoint:TestPoint_Pad_D1.0mm, F.Cu at (352.2, 189.2)
- J801: value Conn_01x04_Socket -> SWD
- J901: value Conn_01x08_Socket -> LCD
- moved C402 6.90 mm to (93.0, 54.9)
- moved R401 6.90 mm to (89.5, 54.9)
- moved R402 6.90 mm to (96.5, 54.9)
- moved U402 6.90 mm to (93.0, 51.4)
- moved U401 2.02 mm to (137.0, 105.2)
- moved C401 2.00 mm to (132.2, 104.2)
Connections:
- U401 pad 2: 5V -> Net-(JP401-C)
- U401 pad 5: unconnected-(U401-PUSH-Pad5) -> /Sensors/ENC__PUSH
Routing:
- net 5V: track 8.51 -> 21.1 mm
- net Net-(JP401-C): track 0.00 -> 6.98 mm
- net /Sensors/ENC__PUSH: track 0.00 -> 4.91 mm
- net /Sensors/ENC__~{CS}: track 0.00 -> 4.89 mm
- net /Sensors/ENC_MISO: track 0.00 -> 4.49 mm
- net /Sensors/ENC_CLK: track 0.00 -> 4.24 mm
- net /Sensors/SDA: track 2.75 -> 4.63 mm
- net /Sensors/SCL: track 2.70 -> 4.56 mm
- net 3.3V: track 19.4 -> 21.2 mm
