File: knobber/knobber.kicad_sch (KiCad schematic)
At the start: 1 part, among them J101 BLDC

Commit message: Updated schematic & PCB
Other:
- sheet Sensors ports: added ENC__PUSH; removed none
Changed lines of the file:
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@@
 	(title_block
 		(title "Knobber")
-		(date "2026-03-14")
+		(date "2026-03-16")
 		(rev "V0.1")
 		(company "Author: Emiel V")
@@
 		)
 		(pin "ENC_MISO" output
-			(at 153.67 39.37 0)
+			(at 153.67 36.83 0)
 			(effects
 				(font
@@
 			)
 		)
+		(pin "ENC__PUSH" output
+			(at 153.67 39.37 0)
+			(effects
+				(font
+					(size 1.27 1.27)
+				)
+				(justify right)
+			)
+		)
